File: hardware/CeilingFanControl/CeilingFanControl(without zones).kicad_pcb (KiCad board)
At the start: 2 copper layers, 60.8 x 61 mm, 28 parts, among them J1 Screw_Terminal_01x02, J2 Conn_01x04, J3 Conn_01x04, J4 Screw_Terminal_01x05, Q1 BTA16-600B, Q2 BTA16-600B, Q3 BTA16-600B, U1 4N25, U2 PIC16F628A-IP, U3 MOC3020M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

Commit message: Commit befora creating tag
Parts:
- moved D4 7.64 mm to (31.0, 62.0), turned to 180 degrees
- moved D3 7.60 mm to (23.4, 65.9), turned to 0 degrees
- moved D1 7.60 mm to (23.4, 58.0), turned to 0 degrees
- moved D2 7.56 mm to (30.9, 54.0), turned to 180 degrees
Connections:
- D2 pad 1: Net-(D1-Pad2) -> Net-(D2-Pad1)
- D2 pad 2: Net-(D2-Pad2) -> Net-(D1-Pad1)
- D3 pad 1: Net-(D1-Pad1) -> Net-(D3-Pad1)
- D3 pad 2: Net-(D3-Pad2) -> Net-(D1-Pad2)
- D4 pad 1: Net-(D3-Pad2) -> Net-(D2-Pad1)
- D4 pad 2: Net-(D2-Pad2) -> Net-(D3-Pad1)
- R1 pad 2: Net-(D1-Pad2) -> Net-(D1-Pad1)
- R2 pad 2: Net-(D3-Pad2) -> Net-(D3-Pad1)
- U1 pad 1: Net-(D2-Pad2) -> Net-(D2-Pad1)
- U1 pad 2: Net-(D1-Pad1) -> Net-(D1-Pad2)
Routing:
- net Net-(D2-Pad2): track 25.1 -> 0.00 mm
- net Net-(D2-Pad1): track 0.00 -> 25.1 mm
- net Net-(D3-Pad2): track 15.0 -> 0.00 mm
- net Net-(D3-Pad1): track 0.00 -> 15.0 mm
- net Net-(D1-Pad2): track 19.6 -> 24.2 mm
- net Net-(D1-Pad1): track 24.2 -> 19.6 mm
